Commit message: refactoring controller to use 6 legs

File: hexapod_description/models/phantomx/urdf/phantomx.xacro (robot description, xacro)
@@ -2,16 +2,4 @@
 <robot name="PhantomX"  xmlns:xacro="http://www.ros.org/wiki/xacro">
   <xacro:include filename="$(find hexapod_description)/models/phantomx/urdf/phantomx.urdf.xacro" />
-  <!-- <xacro:macro name="transmission" params="leg_number joint_number">
-    <transmission name="transmission_${leg_number}_${joint_number}">
-      <type>transmission_interface/SimpleTransmission</type>
-      <joint name="joint_${leg_number}_${joint_number}">
-        <hardwareInterface>hardware_interface::PositionJointInterface</hardwareInterface>
-      </joint>
-      <actuator name="actuator_${leg_number}_${joint_number}">
-        <hardwareInterface>hardware_interface::PositionActuatorInterface</hardwareInterface>
-        <mechanicalReduction>1.0</mechanicalReduction>
-      </actuator>
-    </transmission>
-  </xacro:macro> -->
   <ros2_control name="GazeboSimSystem" type="system">
     <hardware>
@@ -22,7 +10,5 @@
         <command_interface name="position"/>  <!-- controlling joint positions -->
         <command_interface name="velocity"/>  <!-- controlling joint velocities -->
-        <state_interface name="position">
-          <!-- <param name="initial_value">${initial_positions['joint${leg_number}_${joint_number}']}</param> Configuring initial value -->
-        </state_interface>
+        <state_interface name="position"/>
         <state_interface name="velocity"/>
       </joint>

Commit message: joint trajectory controller and kinematic teleportation

File: hexapod_description/models/phantomx/urdf/phantomx.xacro (robot description, xacro)
@@ -48,3 +48,30 @@
     </plugin>
   </gazebo>
+  <xacro:macro name="gazebo_joint" params="leg_number joint_number">
+    <gazebo reference="joint_${leg_number}_${joint_number}">
+      <provideFeedback>true</provideFeedback>
+      <dynamics>
+        <damping>0.1</damping>
+        <friction>0.0</friction>
+      </dynamics>
+    </gazebo>
+  </xacro:macro>
+  <xacro:gazebo_joint leg_number="1" joint_number="1"/>
+  <xacro:gazebo_joint leg_number="1" joint_number="2"/>
+  <xacro:gazebo_joint leg_number="1" joint_number="3"/>
+  <xacro:gazebo_joint leg_number="2" joint_number="1"/>
+  <xacro:gazebo_joint leg_number="2" joint_number="2"/>
+  <xacro:gazebo_joint leg_number="2" joint_number="3"/>
+  <xacro:gazebo_joint leg_number="3" joint_number="1"/>
+  <xacro:gazebo_joint leg_number="3" joint_number="2"/>
+  <xacro:gazebo_joint leg_number="3" joint_number="3"/>
+  <xacro:gazebo_joint leg_number="4" joint_number="1"/>
+  <xacro:gazebo_joint leg_number="4" joint_number="2"/>
+  <xacro:gazebo_joint leg_number="4" joint_number="3"/>
+  <xacro:gazebo_joint leg_number="5" joint_number="1"/>
+  <xacro:gazebo_joint leg_number="5" joint_number="2"/>
+  <xacro:gazebo_joint leg_number="5" joint_number="3"/>
+  <xacro:gazebo_joint leg_number="6" joint_number="1"/>
+  <xacro:gazebo_joint leg_number="6" joint_number="2"/>
+  <xacro:gazebo_joint leg_number="6" joint_number="3"/>
 </robot>
