Commit message: fixed crucial gait bugs

File: hexapod_description/models/phantomx/urdf/phantomx.xacro (robot description, xacro)
@@ -8,10 +8,14 @@
     <xacro:macro name="joint" params="leg_number joint_number">
       <joint name="joint_${leg_number}_${joint_number}">
+        <!-- must stay consistent with <limit effort="2.8"> in phantomx.urdf.xacro:
+             ros2_control saturates commands to this range, so a tighter clamp here
+             silently under-actuates the robot -->
         <command_interface name="effort">
-          <param name="min">-0.5</param>
-          <param name="max">0.5</param>
+          <param name="min">-2.8</param>
+          <param name="max">2.8</param>
         </command_interface>
         <state_interface name="position"/>
         <state_interface name="velocity"/>
+        <state_interface name="effort"/>
       </joint>
     </xacro:macro>
