Commit message: crude hack with feedback action cancelling

File: hexapod_description/models/phantomx/urdf/phantomx.urdf.xacro (robot description, xacro)
@@ -7,9 +7,10 @@
   </joint>
   <joint name="joint_1_1" type="revolute">
-    <limit lower="-2.61799" upper="2.61799" effort="2.80000" velocity="5.65487"/>
+    <limit lower="-2.61799" upper="2.61799" effort="2.8" velocity="5.65487"/>
     <origin rpy="-3.14147 -1.57071 -0.78578" xyz="0.12480 0.06164 0.00112"/>
     <parent link="body"/>
     <child link="coxa1_lf"/>
     <axis xyz="1.00000 0.00000 0.00000"/>
+    <dynamics damping="0.05" friction="0.0"/>
   </joint>
   <joint name="joint_3_coxa" type="fixed">
@@ -19,23 +20,26 @@
   </joint>
   <joint name="joint_3_2" type="revolute">
-    <limit lower="-2.61799" upper="2.61799" effort="2.80000" velocity="5.65487"/>
+    <limit lower="-2.61799" upper="2.61799" effort="2.8" velocity="5.65487"/>
     <origin rpy="3.14159 0.00000 0.00000" xyz="-0.00000 -0.00000 0.00000"/>
     <parent link="coxa2_lr"/>
     <child link="femur_lr"/>
     <axis xyz="1.00000 0.00000 0.00000"/>
+    <dynamics damping="0.05" friction="0.0"/>
   </joint>
   <joint name="joint_3_3" type="revolute">
-    <limit lower="-2.61799" upper="2.61799" effort="2.80000" velocity="5.65487"/>
+    <limit lower="-2.61799" upper="2.61799" effort="2.8" velocity="5.65487"/>
     <origin rpy="-1.57070 -0.00000 3.14159" xyz="-0.00000 -0.06450 -0.01450"/>
     <parent link="femur_lr"/>
     <child link="tibia_lr"/>
     <axis xyz="1.00000 0.00000 0.00000"/>
+    <dynamics damping="0.05" friction="0.0"/>
   </joint>
   <joint name="joint_4_1" type="revolute">
-    <limit lower="-2.61799" upper="2.61799" effort="2.80000" velocity="5.65487"/>
+    <limit lower="-2.61799" upper="2.61799" effort="2.8" velocity="5.65487"/>
     <origin rpy="-3.14147 -1.57071 2.35633" xyz="-0.12480 -0.06164 0.00112"/>
     <parent link="body"/>
     <child link="coxa1_rr"/>
     <axis xyz="1.00000 0.00000 0.00000"/>
+    <dynamics damping="0.05" friction="0.0"/>
   </joint>
   <joint name="joint_4_coxa" type="fixed">
@@ -45,23 +49,26 @@
   </joint>
   <joint name="joint_4_2" type="revolute">
-    <limit lower="-2.61799" upper="2.61799" effort="2.80000" velocity="5.65487"/>
+    <limit lower="-2.61799" upper="2.61799" effort="2.8" velocity="5.65487"/>
     <origin rpy="3.14159 -0.00000 0.00000" xyz="0.00000 0.00000 -0.00000"/>
     <parent link="coxa2_rr"/>
     <child link="femur_rr"/>
     <axis xyz="1.00000 0.00000 0.00000"/>
+    <dynamics damping="0.05" friction="0.0"/>
   </joint>
   <joint name="joint_4_3" type="revolute">
-    <limit lower="-2.61799" upper="2.61799" effort="2.80000" velocity="5.65487"/>
+    <limit lower="-2.61799" upper="2.61799" effort="2.8" velocity="5.65487"/>
     <origin rpy="-1.57070 0.00000 3.14159" xyz="0.00000 -0.06450 -0.01450"/>
     <parent link="femur_rr"/>
     <child link="tibia_rr"/>
     <axis xyz="1.00000 0.00000 0.00000"/>
+    <dynamics damping="0.05" friction="0.0"/>
   </joint>
   <joint name="joint_5_1" type="revolute">
-    <limit lower="-2.61799" upper="2.61799" effort="2.80000" velocity="5.65487"/>
+    <limit lower="-2.61799" upper="2.61799" effort="2.8" velocity="5.65487"/>
     <origin rpy="3.14159 -1.57071 3.14159" xyz="0.00000 -0.10340 0.00112"/>
     <parent link="body"/>
     <child link="coxa1_rm"/>
     <axis xyz="1.00000 0.00000 0.00000"/>
+    <dynamics damping="0.05" friction="0.0"/>
   </joint>
   <joint name="joint_5_coxa" type="fixed">
@@ -71,9 +78,10 @@
   </joint>
   <joint name="joint_5_2" type="revolute">
-    <limit lower="-2.61799" upper="2.61799" effort="2.80000" velocity="5.65487"/>
+    <limit lower="-2.61799" upper="2.61799" effort="2.8" velocity="5.65487"/>
     <origin rpy="3.14159 -0.00000 0.00000" xyz="-0.00000 0.00000 -0.00000"/>
     <parent link="coxa2_rm"/>
     <child link="femur_rm"/>
     <axis xyz="1.00000 0.00000 0.00000"/>
+    <dynamics damping="0.05" friction="0.0"/>
   </joint>
   <joint name="joint_1_coxa" type="fixed">
@@ -83,16 +91,18 @@
   </joint>
   <joint name="joint_5_3" type="revolute">
-    <limit lower="-2.61799" upper="2.61799" effort="2.80000" velocity="5.65487"/>
+    <limit lower="-2.61799" upper="2.61799" effort="2.8" velocity="5.65487"/>
     <origin rpy="-1.57070 0.00000 3.14159" xyz="-0.00000 -0.06450 -0.01450"/>
     <parent link="femur_rm"/>
     <child link="tibia_rm"/>
     <axis xyz="1.00000 0.00000 0.00000"/>
+    <dynamics damping="0.05" friction="0.0"/>
   </joint>
   <joint name="joint_6_1" type="revolute">
-    <limit lower="-2.61799" upper="2.61799" effort="2.80000" velocity="5.65487"/>
+    <limit lower="-2.61799" upper="2.61799" effort="2.8" velocity="5.65487"/>
     <origin rpy="3.14147 -1.57071 -2.35633" xyz="0.12480 -0.06164 0.00112"/>
     <parent link="body"/>
     <child link="coxa1_rf"/>
     <axis xyz="1.00000 0.00000 0.00000"/>
+    <dynamics damping="0.05" friction="0.0"/>
   </joint>
   <joint name="joint_6_coxa" type="fixed">
@@ -102,37 +112,42 @@
   </joint>
   <joint name="joint_6_2" type="revolute">
-    <limit lower="-2.61799" upper="2.61799" effort="2.80000" velocity="5.65487"/>
+    <limit lower="-2.61799" upper="2.61799" effort="2.8" velocity="5.65487"/>
     <origin rpy="3.14159 -0.00000 -0.00000" xyz="-0.00000 0.00000 0.00000"/>
     <parent link="coxa2_rf"/>
     <child link="femur_rf"/>
     <axis xyz="1.00000 0.00000 0.00000"/>
+    <dynamics damping="0.05" friction="0.0"/>
   </joint>
   <joint name="joint_6_3" type="revolute">
-    <limit lower="-2.61799" upper="2.61799" effort="2.80000" velocity="5.65487"/>
+    <limit lower="-2.61799" upper="2.61799" effort="2.8" velocity="5.65487"/>
     <origin rpy="-1.57070 0.00000 3.14159" xyz="-0.00000 -0.06450 -0.01450"/>
     <parent link="femur_rf"/>
     <child link="tibia_rf"/>
     <axis xyz="1.00000 0.00000 0.00000"/>
+    <dynamics damping="0.05" friction="0.0"/>
   </joint>
   <joint name="joint_1_2" type="revolute">
-    <limit lower="-2.61799" upper="2.61799" effort="2.80000" velocity="5.65487"/>
+    <limit lower="-2.61799" upper="2.61799" effort="2.8" velocity="5.65487"/>
     <origin rpy="3.14159 0.00000 0.00000" xyz="0.00000 0.00000 -0.00000"/>
     <parent link="coxa2_lf"/>
     <child link="femur_lf"/>
     <axis xyz="1.00000 0.00000 0.00000"/>
+    <dynamics damping="0.05" friction="0.0"/>
   </joint>
   <joint name="joint_1_3" type="revolute">
-    <limit lower="-2.61799" upper="2.61799" effort="2.80000" velocity="5.65487"/>
+    <limit lower="-2.61799" upper="2.61799" effort="2.8" velocity="5.65487"/>
     <origin rpy="-1.57070 0.00000 3.14159" xyz="0.00000 -0.06450 -0.01450"/>
     <parent link="femur_lf"/>
     <child link="tibia_lf"/>
     <axis xyz="1.00000 0.00000 0.00000"/>
+    <dynamics damping="0.05" friction="0.0"/>
   </joint>
   <joint name="joint_2_1" type="revolute">
-    <limit lower="-2.61799" upper="2.61799" effort="2.80000" velocity="5.65487"/>
+    <limit lower="-2.61799" upper="2.61799" effort="2.8" velocity="5.65487"/>
     <origin rpy="-3.14159 -1.57071 -0.00000" xyz="0.00000 0.10340 0.00112"/>
     <parent link="body"/>
     <child link="coxa1_lm"/>
     <axis xyz="1.00000 0.00000 0.00000"/>
+    <dynamics damping="0.05" friction="0.0"/>
   </joint>
   <joint name="joint_2_coxa" type="fixed">
@@ -142,23 +157,26 @@
   </joint>
   <joint name="joint_2_2" type="revolute">
-    <limit lower="-2.61799" upper="2.61799" effort="2.80000" velocity="5.65487"/>
+    <limit lower="-2.61799" upper="2.61799" effort="2.8" velocity="5.65487"/>
     <origin rpy="3.14159 0.00000 -0.00000" xyz="-0.00000 0.00000 -0.00000"/>
     <parent link="coxa2_lm"/>
     <child link="femur_lm"/>
     <axis xyz="1.00000 0.00000 0.00000"/>
+    <dynamics damping="0.05" friction="0.0"/>
   </joint>
   <joint name="joint_2_3" type="revolute">
-    <limit lower="-2.61799" upper="2.61799" effort="2.80000" velocity="5.65487"/>
+    <limit lower="-2.61799" upper="2.61799" effort="2.8" velocity="5.65487"/>
     <origin rpy="-1.57070 0.00000 3.14159" xyz="-0.00000 -0.06450 -0.01450"/>
     <parent link="femur_lm"/>
     <child link="tibia_lm"/>
     <axis xyz="1.00000 0.00000 0.00000"/>
+    <dynamics damping="0.05" friction="0.0"/>
   </joint>
   <joint name="joint_3_1" type="revolute">
-    <limit lower="-2.61799" upper="2.61799" effort="2.80000" velocity="5.65487"/>
+    <limit lower="-2.61799" upper="2.61799" effort="2.8" velocity="5.65487"/>
     <origin rpy="3.14147 -1.57071 0.78578" xyz="-0.12480 0.06164 0.00112"/>
     <parent link="body"/>
     <child link="coxa1_lr"/>
     <axis xyz="1.00000 0.00000 0.00000"/>
+    <dynamics damping="0.05" friction="0.0"/>
   </joint>
   <link name="base_link"/>

File: hexapod_description/models/phantomx/urdf/phantomx.xacro (robot description, xacro)
@@ -8,6 +8,8 @@
     <xacro:macro name="joint" params="leg_number joint_number">
       <joint name="joint_${leg_number}_${joint_number}">
-        <command_interface name="position"/>  <!-- controlling joint positions -->
-        <command_interface name="velocity"/>  <!-- controlling joint velocities -->
+        <command_interface name="effort">
+          <param name="min">-0.5</param>
+          <param name="max">0.5</param>
+        </command_interface>
         <state_interface name="position"/>
         <state_interface name="velocity"/>
@@ -48,30 +50,3 @@
     </plugin>
   </gazebo>
-  <xacro:macro name="gazebo_joint" params="leg_number joint_number">
-    <gazebo reference="joint_${leg_number}_${joint_number}">
-      <provideFeedback>true</provideFeedback>
-      <dynamics>
-        <damping>0.1</damping>
-        <friction>0.0</friction>
-      </dynamics>
-    </gazebo>
-  </xacro:macro>
-  <xacro:gazebo_joint leg_number="1" joint_number="1"/>
-  <xacro:gazebo_joint leg_number="1" joint_number="2"/>
-  <xacro:gazebo_joint leg_number="1" joint_number="3"/>
-  <xacro:gazebo_joint leg_number="2" joint_number="1"/>
-  <xacro:gazebo_joint leg_number="2" joint_number="2"/>
-  <xacro:gazebo_joint leg_number="2" joint_number="3"/>
-  <xacro:gazebo_joint leg_number="3" joint_number="1"/>
-  <xacro:gazebo_joint leg_number="3" joint_number="2"/>
-  <xacro:gazebo_joint leg_number="3" joint_number="3"/>
-  <xacro:gazebo_joint leg_number="4" joint_number="1"/>
-  <xacro:gazebo_joint leg_number="4" joint_number="2"/>
-  <xacro:gazebo_joint leg_number="4" joint_number="3"/>
-  <xacro:gazebo_joint leg_number="5" joint_number="1"/>
-  <xacro:gazebo_joint leg_number="5" joint_number="2"/>
-  <xacro:gazebo_joint leg_number="5" joint_number="3"/>
-  <xacro:gazebo_joint leg_number="6" joint_number="1"/>
-  <xacro:gazebo_joint leg_number="6" joint_number="2"/>
-  <xacro:gazebo_joint leg_number="6" joint_number="3"/>
 </robot>
